File: USB_TPM/TPM.sch (EAGLE design)
At the start: 47 parts, among them U1 SAM4S4A, X1 TC2050-NL-MCP-NL, Y1 12MHZ

Commit message: schematic complete, board has 57 airwires
Parts:
- removed FRAME1: FRAME-LEDGER, TPM:FRAME-LEDGER
- added C20: 22uF, TPM:CAPACITOR.0603
- added C21: 2.2uF, TPM:CAPACITOR.0201
- added C22: 10uF, TPM:CAPACITOR.0402
- added C23, C24: (no value), TPM:CAPACITOR.0201
- added L1: 2.2uH, TPM:INDUCTOR0402
- added R10: 4.7, TPM:RESISTOR.0402
- added R11, R12, R13, R14, R15, R9: 100K, TPM:RESISTOR.0201
- added R16, R18, R19, R20, R21: (no value), TPM:RESISTOR.0201
- added R8: 470, TPM:RESISTOR.0402
- added U2: TPS62172, TPM:TPS62172
- added Y2: (no value), TPM:CRYSTALEPSONMC146
- C1, C3: value 2200pF -> 0.1uF
- C7: value 2200pF -> (none)
- R1: value 2.2K -> 825
- R2: value 2.2K -> 3.92K
- R6: value (none) -> 4.7K
- R7: value (none) -> 10K
Connections:
- removed net N$7: U1.NRST, X1.RESET
- new net AES: R19.1, U1.PA1/PGMEN1
- new net ECC: R18.1, U1.PA2/PGMEN2
- new net N$16: D4.C, R18.2
- new net N$17: L1.1, U2.SW
- new net N$18: D1.C, R8.2
- new net N$20: D6.C, R16.2
- new net N$21: D5.C, R19.2
- new net N$22: D2.C, R20.2
- new net N$23: D3.C, R21.2
- new net SHA: R16.1, U1.PA0/PGMEN0
- new net STAT0: R20.1, U1.PB0/AD4
- new net STAT1: R21.1, U1.PB1/AD5
- new net VUSB: C21.1, C22.1, R10.2, U2.EN, U2.VIN
- new net XIN32: C23.1, U1.PA7/XIN32/PGMNVALID, Y2.2
- new net XOUT32: C24.1, U1.PA8/XOUT32/PGMM0, Y2.1
- net 3.3V: now also C20.1, D1.A, D2.A, D3.A, D4.A, D5.A, D6.A, L1.2, R11.1, R12.1, R13.1, R14.1, R15.2, R9.2, TPM1.NBO@5, U2.VOS; no longer C7.2
- net CS: now also R15.1
- net GND: now also C20.2, C21.2, C22.2, C23.2, C24.2, C7.2, R8.1, U2.AGND, U2.FB, U2.PAD, U2.PGND; no longer C7.1
- net N$13: now also R10.1
- net N$15: now also TPM1.GPIO-EXPRESS-00
- net N$3: now also R11.2
- net N$4: now also R14.2
- net N$5: now also R12.2
- net N$6: now also R13.2
- net RST: now also C7.1, R9.1, U1.NRST, X1.RESET
Other:
- note added: "32KHz Crystal"
- note added: "CryptoAuthenication ICs"
- note added: "JTAG"
- note added: "Microcontroller"
- note added: "Power Decoupling"
- note added: "Trusted Platform Module"
- note added: "Voltage Regulator"
- moved on the sheet: C1, C10, C11, C12, C13, C14, C15, C16, C17, C18, C19, C2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

Commit message: initial github commit
Parts:
- removed C15: .1uF, TPM:CAPACITOR.0201
- removed C21: 2.2uF, TPM:CAPACITOR.0201
- C23, C24: value (none) -> 22pF
- C5: value (none) -> 0.1uF
- C7: value (none) -> 0.02uF
- R16, R18, R19, R20, R21: value (none) -> 470
- R3, R4: value 27 Ohm -> 27
- R5: value (none) -> 4.7K
- Y2: value (none) -> 32KHz
Connections:
- net 1.2V: no longer C15.1
- net GND: no longer C15.2, C21.2
- net SCL: now also U1.PA4/PGMNCMD
- net SDA: now also U1.PA3
- net VUSB: no longer C21.1
Changed lines of the file:
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@@
 <part name="SUPPLY8" library="TPM" deviceset="3.3V" device=""/>
 <part name="SUPPLY9" library="TPM" deviceset="3.3V" device=""/>
-<part name="R3" library="TPM" deviceset="RESISTOR" device=".0402" value="27  Ohm"/>
-<part name="R4" library="TPM" deviceset="RESISTOR" device=".0402" value="27 Ohm"/>
+<part name="R3" library="TPM" deviceset="RESISTOR" device=".0402" value="27"/>
+<part name="R4" library="TPM" deviceset="RESISTOR" device=".0402" value="27"/>
 <part name="SUPPLY10" library="TPM" deviceset="1.2V" device=""/>
 <part name="SUPPLY11" library="TPM" deviceset="3.3V" device=""/>
-<part name="C5" library="TPM" deviceset="CAPACITOR" device=".0201"/>
+<part name="C5" library="TPM" deviceset="CAPACITOR" device=".0201" value="0.1uF"/>
 <part name="GND13" library="TPM" deviceset="GND" device=""/>
 <part name="C9" library="TPM" deviceset="CAPACITOR" device=".0201" value=".1uF"/>
@@
 <part name="C13" library="TPM" deviceset="CAPACITOR" device=".0201" value=".1uF"/>
 <part name="C14" library="TPM" deviceset="CAPACITOR" device=".0201" value=".1uF"/>
-<part name="C15" library="TPM" deviceset="CAPACITOR" device=".0201" value=".1uF"/>
 <part name="C16" library="TPM" deviceset="CAPACITOR" device=".0201" value=".1uF"/>
 <part name="C17" library="TPM" deviceset="CAPACITOR" device=".0402" value="4.7uF"/>
@@
 <part name="C6" library="TPM" deviceset="CAPACITOR" device=".0201" value="2200pF"/>
 <part name="Y1" library="TPM" deviceset="RESONATOR" device="12MHZ" value="12MHZ"/>
-<part name="R5" library="TPM" deviceset="RESISTOR" device=".0201"/>
+<part name="R5" library="TPM" deviceset="RESISTOR" device=".0201" value="4.7K"/>
 <part name="R6" library="TPM" deviceset="RESISTOR" device=".0201" value="4.7K"/>
 <part name="R7" library="TPM" deviceset="RESISTOR" device=".0201" value="10K"/>
@@
 <part name="R8" library="TPM" deviceset="RESISTOR" device=".0402" value="470"/>
 <part name="R9" library="TPM" deviceset="RESISTOR" device=".0201" value="100K"/>
-<part name="C7" library="TPM" deviceset="CAPACITOR" device=".0201"/>
+<part name="C7" library="TPM" deviceset="CAPACITOR" device=".0201" value="0.02uF"/>
 <part name="GND20" library="TPM" deviceset="GND" device=""/>
 <part name="SUPPLY17" library="TPM" deviceset="3.3V" device=""/>
@@
 <part name="R10" library="TPM" deviceset="RESISTOR" device=".0402" value="4.7"/>
 <part name="SUPPLY18" library="TPM" deviceset="VUSB" device=""/>
-<part name="C21" library="TPM" deviceset="CAPACITOR" device=".0201" value="2.2uF"/>
-<part name="Y2" library="TPM" deviceset="CRYSTAL" device="EPSONMC146"/>
+<part name="Y2" library="TPM" deviceset="CRYSTAL" device="EPSONMC146" value="32KHz"/>
 <part name="C22" library="TPM" deviceset="CAPACITOR" device=".0402" value="10uF"/>
 <part name="SUPPLY19" library="TPM" deviceset="VUSB" device=""/>
@@
 <part name="R15" library="TPM" deviceset="RESISTOR" device=".0201" value="100K"/>
 <part name="SUPPLY21" library="TPM" deviceset="3.3V" device=""/>
-<part name="C23" library="TPM" deviceset="CAPACITOR" device=".0201"/>
-<part name="C24" library="TPM" deviceset="CAPACITOR" device=".0201"/>
+<part name="C23" library="TPM" deviceset="CAPACITOR" device=".0201" value="22pF"/>
+<part name="C24" library="TPM" deviceset="CAPACITOR" device=".0201" value="22pF"/>
 <part name="GND22" library="TPM" deviceset="GND" device=""/>
-<part name="R16" library="TPM" deviceset="RESISTOR" device=".0201"/>
-<part name="R18" library="TPM" deviceset="RESISTOR" device=".0201"/>
-<part name="R19" library="TPM" deviceset="RESISTOR" device=".0201"/>
-<part name="R20" library="TPM" deviceset="RESISTOR" device=".0201"/>
-<part name="R21" library="TPM" deviceset="RESISTOR" device=".0201"/>
+<part name="R16" library="TPM" deviceset="RESISTOR" device=".0201" value="470"/>
+<part name="R18" library="TPM" deviceset="RESISTOR" device=".0201" value="470"/>
+<part name="R19" library="TPM" deviceset="RESISTOR" device=".0201" value="470"/>
+<part name="R20" library="TPM" deviceset="RESISTOR" device=".0201" value="470"/>
+<part name="R21" library="TPM" deviceset="RESISTOR" device=".0201" value="470"/>
 <part name="SUPPLY22" library="TPM" deviceset="3.3V" device=""/>
 <part name="SUPPLY23" library="TPM" deviceset="3.3V" device=""/>
@@
 <instance part="SUPPLY9" gate="G$1" x="279.4" y="73.66"/>
 <instance part="R3" gate="G$1" x="63.5" y="109.22" smashed="yes">
-<attribute name="NAME" x="59.69" y="105.6386" size="1.778" layer="95"/>
-<attribute name="VALUE" x="64.77" y="105.918" size="1.778" layer="96"/>
+<attribute name="NAME" x="64.77" y="105.6386" size="1.778" layer="95"/>
+<attribute name="VALUE" x="64.77" y="103.378" size="1.778" layer="96"/>
 </instance>
 <instance part="R4" gate="G$1" x="63.5" y="111.76" smashed="yes">
-<attribute name="NAME" x="59.69" y="113.2586" size="1.778" layer="95"/>
+<attribute name="NAME" x="64.77" y="115.7986" size="1.778" layer="95"/>
 <attribute name="VALUE" x="64.77" y="113.538" size="1.778" layer="96"/>
 </instance>
@@
 <instance part="C13" gate="G$1" x="340.36" y="177.8"/>
 <instance part="C14" gate="G$1" x="350.52" y="177.8"/>
-<instance part="C15" gate="G$1" x="360.68" y="177.8"/>
 <instance part="C16" gate="G$1" x="340.36" y="205.74"/>
 <instance part="C17" gate="G$1" x="350.52" y="205.74"/>
@@
 <instance part="R10" gate="G$1" x="50.8" y="129.54" rot="R90"/>
 <instance part="SUPPLY18" gate="G$1" x="50.8" y="142.24"/>
-<instance part="C21" gate="G$1" x="55.88" y="134.62"/>
 <instance part="Y2" gate="G$1" x="147.32" y="243.84" rot="R180"/>
 <instance part="C22" gate="G$1" x="27.94" y="236.22"/>
@@
 <wire x1="55.88" y1="127" x2="55.88" y2="116.84" width="0.1524" layer="91"/>
 <junction x="55.88" y="116.84"/>
-<pinref part="C21" gate="G$1" pin="2"/>
-<wire x1="55.88" y1="129.54" x2="55.88" y2="127" width="0.1524" layer="91"/>
-<junction x="55.88" y="127"/>
 </segment>
 <segment>
@@
 <wire x1="340.36" y1="170.18" x2="350.52" y2="170.18" width="0.1524" layer="91"/>
 <wire x1="350.52" y1="170.18" x2="350.52" y2="172.72" width="0.1524" layer="91"/>
-<pinref part="C15" gate="G$1" pin="2"/>
-<wire x1="350.52" y1="170.18" x2="360.68" y2="170.18" width="0.1524" layer="91"/>
-<wire x1="360.68" y1="170.18" x2="360.68" y2="172.72" width="0.1524" layer="91"/>
 <junction x="340.36" y="170.18"/>
-<junction x="350.52" y="170.18"/>
 </segment>
 <segment>
@@
 <wire x1="271.78" y1="53.34" x2="271.78" y2="60.96" width="0.1524" layer="91"/>
 <junction x="271.78" y="53.34"/>
+</segment>
+<segment>
+<pinref part="U1" gate="G$1" pin="PA3"/>
+<wire x1="152.4" y1="165.1" x2="157.48" y2="165.1" width="0.1524" layer="91" style="longdash"/>
+<label x="157.48" y="165.1" size="1.4224" layer="95" font="vector" ratio="12" xref="yes"/>
 </segment>
 </net>
@@
 <junction x="279.4" y="48.26"/>
 </segment>
+<segment>
+<pinref part="U1" gate="G$1" pin="PA4/PGMNCMD"/>
+<wire x1="152.4" y1="162.56" x2="157.48" y2="162.56" width="0.1524" layer="91" style="longdash"/>
+<label x="157.48" y="162.56" size="1.4224" layer="95" font="vector" ratio="12" xref="yes"/>
+</segment>
 </net>
 <net name="3.3V" class="0">
@@
 <wire x1="350.52" y1="180.34" x2="350.52" y2="182.88" width="0.1524" layer="91"/>
 <wire x1="350.52" y1="182.88" x2="340.36" y2="182.88" width="0.1524" layer="91"/>
-<pinref part="C15" gate="G$1" pin="1"/>
-<wire x1="360.68" y1="180.34" x2="360.68" y2="182.88" width="0.1524" layer="91"/>
-<wire x1="360.68" y1="182.88" x2="350.52" y2="182.88" width="0.1524" layer="91"/>
 <junction x="340.36" y="182.88"/>
-<junction x="350.52" y="182.88"/>
 </segment>
 </net>
@@
 </segment>
 <segment>
-<pinref part="U1" gate="G$1" pin="NRST"/>
-<wire x1="152.4" y1="116.84" x2="160.02" y2="116.84" width="0.1524" layer="91"/>
-<wire x1="160.02" y1="116.84" x2="167.64" y2="116.84" width="0.1524" layer="91"/>
 <wire x1="167.64" y1="116.84" x2="167.64" y2="88.9" width="0.1524" layer="91"/>
 <wire x1="167.64" y1="88.9" x2="93.98" y2="88.9" width="0.1524" layer="91"/>
@@
 <pinref part="X1" gate="G$1" pin="RESET"/>
 <wire x1="93.98" y1="45.72" x2="96.52" y2="45.72" width="0.1524" layer="91"/>
+<pinref part="R9" gate="G$1" pin="1"/>
 <pinref part="C7" gate="G$1" pin="1"/>
 <wire x1="160.02" y1="114.3" x2="160.02" y2="116.84" width="0.1524" layer="91"/>
-<pinref part="R9" gate="G$1" pin="1"/>
+<pinref part="U1" gate="G$1" pin="NRST"/>
 <wire x1="160.02" y1="116.84" x2="160.02" y2="119.38" width="0.1524" layer="91"/>
+<wire x1="152.4" y1="116.84" x2="160.02" y2="116.84" width="0.1524" layer="91" style="longdash"/>
+<wire x1="160.02" y1="116.84" x2="167.64" y2="116.84" width="0.1524" layer="91" style="longdash"/>
 <junction x="160.02" y="116.84"/>
 </segment>
@@
 <pinref part="R10" gate="G$1" pin="2"/>
 <pinref part="SUPPLY18" gate="G$1" pin="VUSB"/>
-<wire x1="50.8" y1="134.62" x2="50.8" y2="137.16" width="0.1524" layer="91"/>
-<pinref part="C21" gate="G$1" pin="1"/>
-<wire x1="50.8" y1="137.16" x2="50.8" y2="142.24" width="0.1524" layer="91"/>
-<wire x1="50.8" y1="137.16" x2="55.88" y2="137.16" width="0.1524" layer="91"/>
-<junction x="50.8" y="137.16"/>
-</segment>
-<segment>
+<wire x1="50.8" y1="134.62" x2="50.8" y2="142.24" width="0.1524" layer="91"/>
+</segment>
+<segment>
