File: Hardware/openTPM-v12.brd (EAGLE design)
At the start: 45 x 19 mm, 65 parts, among them U1 SAM4S4A, U2 TPS62172, X1 TC2050-NL-MCP-NL, Y1 12MHZ, Y2 32KHz

Commit message: reorg of images, update to board trace widths for power, added to gitignore
Parts:
- ECC1: value ATECC108 -> ATECC508
