File: Hardware/openTPM-v37.sch (EAGLE design)
At the start: 62 parts, among them U1 SAM4S4A, U2 TPS62172, U3 TC58CVG0S3HQAIEWSON, Y1 12MHZ, Y2 32KHz

Commit message: OpenTPM v37 upload routing done
Parts:
- removed SL1: SLIDER_PASSIVE_1SEG, u2ftoken:SLIDER_PASSIVE_1SEG
- added 3V3, PB4, PB5, RST, SWCLK, SWDIO: PTR1B1,27, CHEEPER-REV0.51A:PTR1B1,27
- added R11: 10K, TPM:RESISTOR.0402
- U1: value SAM4S4A -> ATSAMD21G18_QFN; device TPM:SAM4S4A -> microbuilder:ATSAMD21G_QFN
Connections:
- removed net N$1: R4.2, U1.DDM/PB10
- removed net N$2: R3.2, U1.DDP/PB11
- removed net N$3: U1.TDI/PB4
- removed net N$4: U1.TDO/TRACESWO/PB5
- removed net N$5: U1.TMS/SWDIO/PB6
- removed net N$6: U1.TCK/SWCLK/PB7
- new net CAP: R11.2
- new net DM: R4.2, U1.PA24/I12/SERCOM3+5.2/D-
- new net DP: R3.2, U1.PA25/I13/SERCOM3+5.3/D+
- new net N$19: U1.PA07/I7/AIN7/SERCOM0.3/I2SD0, U3.CS
- new net N$24: U1.PA05/EINT5/AIN5/SERCOM0.1, U3.HOLD/SO3
- new net N$25: U1.PA06/EINT6/AIN6/SERCOM0.2, U3.WP/SO2
- new net PB08: PB4.TP, U1.PB08/I8/AIN2/SERCOM4.0
- new net PB09: PB5.TP, U1.PB09/I9/AIN3/SERCOM4.1
- new net SLIDE: R11.1, U1.PA21/I5/SERCOM3+5.3/I2SFS0
- new net SWCLK: SWCLK.TP, U1.PA30/I10/SECOM1.2/SWCLK
- new net SWDIO: SWDIO.TP, U1.PA31/I11/SECOM1.3/SWDIO
- net 1.2V: now also U1.VDDCORE; no longer U1.VDDCORE@18, U1.VDDCORE@41, U1.VDDOUT, U1.VDDPLL
- net 3.3V: now also 3V3.TP, U1.VDDA, U1.VDDIO; no longer U1.VDDIO@13, U1.VDDIO@33, U1.VDDIO@47
- net AES: now also U1.PA03/EINT3/VREFA/AIN1; no longer U1.PA1/PGMEN1
- net CLK: now also U1.PB11/I11/SERCOM4.3/I2SCL; no longer U1.PA14/PGMD2
- net CS: now also U1.PA13/I13/I2C/SERCOM2+4.1; no longer U1.PA11/PGMM3
- net ECC: now also U1.PA04/EINT4/VREFB/AIN4/SERCOM0.0; no longer U1.PA2/PGMEN2
- net GND: now also U1.GND, U1.GNDA; no longer U1.GND@2, U1.GND@34
- net MISO: now also U1.PA12/I12/I2C/SERCOM2+4.0; no longer U1.PA12/PGMD0
- net MOSI: now also U1.PB10/I10/SERCOM4.2/I2SMC; no longer U1.PA13/PGMD1
- net N$8: now also U1.PA15/I15/SERCOM2+4.3; no longer U1.XOUT/PB8
- net N$9: now also U1.PA14/I14/SERCOM2+4.2; no longer U1.XIN/PB9/PGMCK
- net RST: now also RST.TP, U1./RESET; no longer U1.NRST
- net SCL: now also U1.PA23/I2C/I7/SERCOM3+5.1/SOF; no longer U1.PA4/PGMNCMD
- net SDA: now also U1.PA22/I2C/I6/SERCOM3+5.0; no longer U1.PA3
- net SHA: now also U1.PA02/EINT2/AIN0/Y0/VOUT; no longer U1.PA0/PGMEN0
- net STAT0: now also U1.PB02/I2/AIN10/SERCOM5.0; no longer U1.PB0/AD4
- net STAT1: now also U1.PB03/I3/AIN11/SERCOM5.1; no longer U1.PB1/AD5
- net XIN32: now also U1.PA00/EINT0/SERCOM1.0; no longer U1.PA7/XIN32/PGMNVALID
- net XOUT32: now also U1.PA01/EINT1/SERCOM1.1; no longer U1.PA8/XOUT32/PGMM0
Other:
- note added: "CAPACTIVE PLANE"
- note removed: "JTAG"
- moved on the sheet: C5, C7, JP1, R10, R15, R3, R4, R9, Y1
